Commit message: fixed settings for Gazebo with Sphero

File: sphero_ros/sphero_description/urdf/sphero.urdf (robot description, URDF)
Before this commit: robot sphero, 1 links, 0 joints
Links:
- link base_link: geometry collision sphere radius=0.0381; visual mesh filename=package://sphero_description/meshes/Sphero_Textured.dae scale=0.8 0.8 0.8
